File: network_player/network_player.kicad_sch (KiCad schematic)
At the start: 76 parts, among them J1 Raspberry_Pi_2_3, J4 USB_C_Receptacle_USB2.0, Q1 BC817, Q2 BC817, Q3 MMBT3904, SW1 SW_Push, SW2 SW_Push, SW3 SW_Push, U1 F1C100s, U3 W25N01GVZEIG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

Commit message: Fully update gerbers before sending again to jlcpcb, also add silkscreen with copyright
Parts:
- U6: footprint Package_DFN_QFN:QFN-20-1EP_3x3mm_P0.45mm_EP1.6x1.6mm -> Package_DFN_QFN:QFN-20-1EP_3x3mm_P0.4mm_EP1.65x1.65mm
Changed lines of the file:
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@@
       (effects (font (size 1.27 1.27)))
     )
-    (property "Footprint" "Package_DFN_QFN:QFN-20-1EP_3x3mm_P0.45mm_EP1.6x1.6mm" (at 68.58 53.975 0)
+    (property "Footprint" "Package_DFN_QFN:QFN-20-1EP_3x3mm_P0.4mm_EP1.65x1.65mm" (at 68.58 53.975 0)
       (effects (font (size 1.27 1.27)) hide)
     )

Commit message: first corrections
Parts:
- added R23, R24: 10k, Resistor_SMD:R_0402_1005Metric, symbol Device:R_Small
- added R25, R26: 0R, Resistor_SMD:R_0402_1005Metric, symbol Device:R_Small
Connections:
- net +3V3: now also R23.2, R24.2
- net +5V: now also U6.18 (EN3), U6.8 (EN2), U6.9 (EN1)
- net DTR: no longer J1.22 (GPIO25)
- net GPIO_9: now also R23.1
- net RTS: no longer J1.37 (GPIO26)
- net SPDIF: now also J1.37 (GPIO26); no longer J1.38 (GPIO20/MOSI1)
- net ESP32_USB_D-: now reaches J1.13 (GPIO27)
- net ESP32_USB_D-: now also U4.26 (GPIO18/USB_D-)
- net I2S_DIN: now reaches U1.44 (PE5/CSI_D2/LCD_D17/DA_IN/EINTE5)
- net I2S_DIN: now also J1.38 (GPIO20/MOSI1)
- net GPIO_8: now reaches U4.22 (GPIO8)
- net GPIO_8: now also R24.1
- net ESP32_USB_D+: now reaches U4.27 (GPIO19/USB_D+)
- net ESP32_USB_D+: now also J1.22 (GPIO25)
- net U0RXD renamed ESP32_RX
- net ESP32_RX: now also R25.1, R26.1; no longer U1.10 (PD4/LCD_D6/UART1_TX/EINTD4)
- net U0TXD renamed ESP32_TX
- net ESP32_TX: no longer U1.9 (PD3/LCD_D5/UART1_RX/EINTD3)
- new net ESP32_RXD: R26.2, U1.10 (PD4/LCD_D6/UART1_TX/EINTD4)
- new net ESP32_TXD: R25.2, U1.9 (PD3/LCD_D5/UART1_RX/EINTD3)
- no-connect marks 31 -> 27

Commit message: recover for v1.1
Parts:
- removed Q1, Q2: BC817, Package_TO_SOT_SMD:SOT-23, symbol Transistor_BJT:BC817
- removed R11, R12, R26: 0R, Resistor_SMD:R_0402_1005Metric, symbol Device:R_Small
- removed R14, R15: 10k, Resistor_SMD:R_0402_1005Metric, symbol Device:R_Small
- D1: LCSC (none) -> C2290
- R25: value 0R -> 10k; LCSC C17168 -> C25744
Connections:
- net ESP32_RXD is gone; now on net U0RXD: U1.10 (PD4/LCD_D6/UART1_TX/EINTD4)
- net +3V3: now also R23.1, R25.1; no longer R23.2, R24.2
- net DTR: now also J1.22 (GPIO25); no longer U1.7 (PD1/LCD_D3/UART1_RTS/EINTD1)
- net GND: now also R24.2
- net RTS: now also J1.37 (GPIO26); no longer U1.8 (PD2/LCD_D4/UART1_CTS/EINTD2)
- net SPDIF: now also J1.38 (GPIO20/MOSI1); no longer J1.37 (GPIO26)
- net SPI_CS: now also U1.26 (PD18/LCD_CLK/SPI0_CS/EINTD18); no longer U1.42 (PE7/CSI_D4/UART2_TX/SPI1_CS/EINTE7)
- net SPI_MISO: now also U1.61 (PC2/SPI0_MISO/SDC1_D0), U3.2 (SO/SIO1); no longer U1.39 (PE10/CSI_D7/UART2_CTS/SPI1_MISO/EINTE10)
- net SPI_MOSI: now also SW2.1, U1.62 (PC3/SPI0_MOSI/UART0_TX), U3.5 (SI/SIO0); no longer U1.41 (PE8/CSI_D5/UART2_RX/SPI1_MOSI/EINTE8)
- net WIFI_HANDSHAKE: now also R23.2
- net WIFI_SPI_CLK: now also U1.40 (PE9/CSI_D6/UART2_RTS/SPI1_CLK/EINTE9); no longer U1.28 (PD20/LCD_HSYNC/SPI0_CLK/EINTD20)
- net WIFI_SPI_CS: now also U1.42 (PE7/CSI_D4/UART2_TX/SPI1_CS/EINTE7); no longer U1.26 (PD18/LCD_CLK/SPI0_CS/EINTD18)
- net WIFI_SPI_MISO: now also U1.39 (PE10/CSI_D7/UART2_CTS/SPI1_MISO/EINTE10); no longer U1.29 (PD21/LCD_VSYNC/SPI0_MISO/EINTD21)
- net WIFI_SPI_MOSI: now also U1.41 (PE8/CSI_D5/UART2_RX/SPI1_MOSI/EINTE8); no longer U1.27 (PD19/LCD_DE/SPI0_MOSI/EINTD19)
- net SPI_MCLK: now reaches U1.59 (PC0/SPI0_CLK/SDC1_CLK), U3.6 (SCLK)
- net SPI_MCLK: now also J1.23 (SCLK0/GPIO11)
- net CHIP_PU renamed ESP_RST
- net ESP_RST: now also U1.7 (PD1/LCD_D3/UART1_RTS/EINTD1)
- net ESP32_RX renamed U0RXD
- net U0RXD: no longer R25.1
- net ESP32_TX renamed U0TXD
- net U0TXD: now also U1.9 (PD3/LCD_D5/UART1_RX/EINTD3)
- net ESP32_TXD renamed ESP_BOOT
- net ESP_BOOT: now also U1.8 (PD2/LCD_D4/UART1_CTS/EINTD2), U4.23 (GPIO9); no longer U1.9 (PD3/LCD_D5/UART1_RX/EINTD3)
- net ESP32_USB_D+: no longer names the net of U4.27 (GPIO19/USB_D+)
- net ESP32_USB_D+: no longer J1.22 (GPIO25)
- net ESP32_USB_D-: no longer names the net of J1.13 (GPIO27)
- net ESP32_USB_D-: no longer U4.26 (GPIO18/USB_D-)
- net GPIO18: no longer names the net of J1.12 (GPIO18/PWM0)
- net GPIO18: no longer U1.79 (LRADC0)
- net GPIO_8: no longer names the net of R24.1, U4.22 (GPIO8)
- removed net GPIO_9: R23.1, SW2.1, U4.23 (GPIO9)
- net I2S_DIN: no longer names the net of U1.44 (PE5/CSI_D2/LCD_D17/DA_IN/EINTE5)
- net I2S_DIN: no longer J1.38 (GPIO20/MOSI1)
- removed net SPI_CLK: J1.23 (SCLK0/GPIO11), U1.40 (PE9/CSI_D6/UART2_RTS/SPI1_CLK/EINTE9)
- no-connect marks 27 -> 38
